Commit message: new model

File: robots/msl_skycrane.URDF (robot description, URDF)
Before this commit: robot msl_skycrane, 6 links, 5 joints
Links:
- removed link bot_plate
- removed link left_down_arm
- removed link left_upper_arm
- removed link right_down_arm
- removed link right_upper_arm
- added link arm_0, mass 2089.2; collision mesh filename=package://msl_skycrane_description/meshes/arm_0.STL; visual mesh filename=package://msl_skycrane_description/meshes/arm_0.STL
- added link arm_1, mass 2089.22272867894; collision mesh filename=package://msl_skycrane_description/meshes/arm_1.STL; visual mesh filename=package://msl_skycrane_description/meshes/arm_1.STL
- added link arm_2, mass 2089.22272867895; collision mesh filename=package://msl_skycrane_description/meshes/arm_2.STL; visual mesh filename=package://msl_skycrane_description/meshes/arm_2.STL
- added link arm_3, mass 2089.22272867894; collision mesh filename=package://msl_skycrane_description/meshes/arm_3.STL; visual mesh filename=package://msl_skycrane_description/meshes/arm_3.STL
- added link elbow_00, mass 3.036; collision mesh filename=package://msl_skycrane_description/meshes/elbow_00.STL; visual mesh filename=package://msl_skycrane_description/meshes/elbow_00.STL
- added link elbow_01, mass 3.036; collision mesh filename=package://msl_skycrane_description/meshes/elbow_01.STL; visual mesh filename=package://msl_skycrane_description/meshes/elbow_01.STL
- added link elbow_10, mass 3.036; collision mesh filename=package://msl_skycrane_description/meshes/elbow_10.STL; visual mesh filename=package://msl_skycrane_description/meshes/elbow_10.STL
- added link elbow_11, mass 3.036; collision mesh filename=package://msl_skycrane_description/meshes/elbow_11.STL; visual mesh filename=package://msl_skycrane_description/meshes/elbow_11.STL
- added link elbow_20, mass 3.03601604481673; collision mesh filename=package://msl_skycrane_description/meshes/elbow_20.STL; visual mesh filename=package://msl_skycrane_description/meshes/elbow_20.STL
- added link elbow_21, mass 3.03601604481672; collision mesh filename=package://msl_skycrane_description/meshes/elbow_21.STL; visual mesh filename=package://msl_skycrane_description/meshes/elbow_21.STL
- added link elbow_30, mass 3.03601604481672; collision mesh filename=package://msl_skycrane_description/meshes/elbow_30.STL; visual mesh filename=package://msl_skycrane_description/meshes/elbow_30.STL
- added link elbow_31, mass 3.03601604481672; collision mesh filename=package://msl_skycrane_description/meshes/elbow_31.STL; visual mesh filename=package://msl_skycrane_description/meshes/elbow_31.STL
- added link engine_00, mass 793.36; collision mesh filename=package://msl_skycrane_description/meshes/engine_00.STL; visual mesh filename=package://msl_skycrane_description/meshes/engine_00.STL
- added link engine_01, mass 793.36; collision mesh filename=package://msl_skycrane_description/meshes/engine_01.STL; visual mesh filename=package://msl_skycrane_description/meshes/engine_01.STL
- added link engine_10, mass 793.36; collision mesh filename=package://msl_skycrane_description/meshes/engine_10.STL; visual mesh filename=package://msl_skycrane_description/meshes/engine_10.STL
- added link engine_11, mass 793.36; collision mesh filename=package://msl_skycrane_description/meshes/engine_11.STL; visual mesh filename=package://msl_skycrane_description/meshes/engine_11.STL
- added link engine_20, mass 793.355843738094; collision mesh filename=package://msl_skycrane_description/meshes/engine_20.STL; visual mesh filename=package://msl_skycrane_description/meshes/engine_20.STL
- added link engine_21, mass 793.355843738093; collision mesh filename=package://msl_skycrane_description/meshes/engine_21.STL; visual mesh filename=package://msl_skycrane_description/meshes/engine_21.STL
- added link engine_30, mass 793.355843738094; collision mesh filename=package://msl_skycrane_description/meshes/engine_30.STL; visual mesh filename=package://msl_skycrane_description/meshes/engine_30.STL
- added link engine_31, mass 793.355843738094; collision mesh filename=package://msl_skycrane_description/meshes/engine_31.STL; visual mesh filename=package://msl_skycrane_description/meshes/engine_31.STL
- added link shoulder_00, mass 8.0556; collision mesh filename=package://msl_skycrane_description/meshes/shoulder_00.STL; visual mesh filename=package://msl_skycrane_description/meshes/shoulder_00.STL
- added link shoulder_01, mass 8.0556; collision mesh filename=package://msl_skycrane_description/meshes/shoulder_01.STL; visual mesh filename=package://msl_skycrane_description/meshes/shoulder_01.STL
- added link shoulder_10, mass 8.0556; collision mesh filename=package://msl_skycrane_description/meshes/shoulder_10.STL; visual mesh filename=package://msl_skycrane_description/meshes/shoulder_10.STL
- added link shoulder_11, mass 8.0556; collision mesh filename=package://msl_skycrane_description/meshes/shoulder_11.STL; visual mesh filename=package://msl_skycrane_description/meshes/shoulder_11.STL
- added link shoulder_20, mass 8.05560156812752; collision mesh filename=package://msl_skycrane_description/meshes/shoulder_20.STL; visual mesh filename=package://msl_skycrane_description/meshes/shoulder_20.STL
- added link shoulder_21, mass 8.05560156812752; collision mesh filename=package://msl_skycrane_description/meshes/shoulder_21.STL; visual mesh filename=package://msl_skycrane_description/meshes/shoulder_21.STL
- added link shoulder_30, mass 8.05560156812752; collision mesh filename=package://msl_skycrane_description/meshes/shoulder_30.STL; visual mesh filename=package://msl_skycrane_description/meshes/shoulder_30.STL
- added link shoulder_31, mass 8.05560156812752; collision mesh filename=package://msl_skycrane_description/meshes/shoulder_31.STL; visual mesh filename=package://msl_skycrane_description/meshes/shoulder_31.STL
- added link top_plate, mass 794.77; collision mesh filename=package://msl_skycrane_description/meshes/top_plate.STL; visual mesh filename=package://msl_skycrane_description/meshes/top_plate.STL
- added link wrist_00, mass 2.6791; collision mesh filename=package://msl_skycrane_description/meshes/wrist_00.STL; visual mesh filename=package://msl_skycrane_description/meshes/wrist_00.STL
- added link wrist_01, mass 2.6791; collision mesh filename=package://msl_skycrane_description/meshes/wrist_01.STL; visual mesh filename=package://msl_skycrane_description/meshes/wrist_01.STL
- added link wrist_10, mass 2.6791; collision mesh filename=package://msl_skycrane_description/meshes/wrist_10.STL; visual mesh filename=package://msl_skycrane_description/meshes/wrist_10.STL
- added link wrist_11, mass 2.6791; collision mesh filename=package://msl_skycrane_description/meshes/wrist_11.STL; visual mesh filename=package://msl_skycrane_description/meshes/wrist_11.STL
- added link wrist_20, mass 2.67913313983108; collision mesh filename=package://msl_skycrane_description/meshes/wrist_20.STL; visual mesh filename=package://msl_skycrane_description/meshes/wrist_20.STL
- added link wrist_21, mass 2.67913313983112; collision mesh filename=package://msl_skycrane_description/meshes/wrist_21.STL; visual mesh filename=package://msl_skycrane_description/meshes/wrist_21.STL
- added link wrist_30, mass 2.67912524460953; collision mesh filename=package://msl_skycrane_description/meshes/wrist_30.STL; visual mesh filename=package://msl_skycrane_description/meshes/wrist_30.STL
- added link wrist_31, mass 2.67912524460955; collision mesh filename=package://msl_skycrane_description/meshes/wrist_31.STL; visual mesh filename=package://msl_skycrane_description/meshes/wrist_31.STL
- link base_link: mass 101.141220442297 -> 85.813; geometry collision mesh filename=package://msl_skycrane_description/meshes/base_link.STL; visual mesh filename=package://msl_skycrane_description/meshes/base_link.STL
Joints:
- removed joint bot_plate_joint
- removed joint left_down_arm_joint
- removed joint left_upper_arm_joint
- removed joint right_down_arm_joint
- removed joint right_upper_arm_joint
- added joint arm_0_joint: type fixed, parent top_plate, child arm_0, origin xyz=-0.111602540378444 -2 -1.50669872981078 rpy=0 1.04719755119662 0, axis 0 0 0
- added joint arm_1_joint: type fixed, parent top_plate, child arm_1, origin xyz=1.249 -2 -0.85 rpy=0 0 0, axis 0 0 0
- added joint arm_2_joint: type fixed, parent top_plate, child arm_2, origin xyz=0.1116 -2 1.5067 rpy=3.1416 -1.0472 3.1416, axis 0 0 0
- added joint arm_3_joint: type fixed, parent top_plate, child arm_3, origin xyz=-1.249 -2 0.85 rpy=3.1416 0 3.1416, axis 0 0 0
- added joint elbow_00_joint: type fixed, parent shoulder_00, child elbow_00, origin xyz=0 0 0 rpy=1.5708 1.0472 2.2093E-14, axis 0 0 0
- added joint elbow_01_joint: type fixed, parent shoulder_01, child elbow_01, origin xyz=0 0 0 rpy=1.5708 1.0472 2.2093E-14, axis 0 0 0
- added joint elbow_10_joint: type fixed, parent shoulder_10, child elbow_10, origin xyz=0 0 0 rpy=1.5708 1.0472 0, axis 0 0 0
- added joint elbow_11_joint: type fixed, parent shoulder_11, child elbow_11, origin xyz=0 0 0 rpy=1.5708 1.0472 0, axis 0 0 0
- added joint elbow_20_joint: type fixed, parent shoulder_20, child elbow_20, origin xyz=0.20321 0 0.40196 rpy=-1.5708 1.0472 2.2093E-14, axis 0 0 0
- added joint elbow_21_joint: type fixed, parent shoulder_21, child elbow_21, origin xyz=0 0 0 rpy=1.5708 -1.0472 -3.1416, axis 0 0 0
- added joint elbow_30_joint: type fixed, parent shoulder_30, child elbow_30, origin xyz=0 0 0 rpy=1.5708 -1.0472 3.1416, axis 0 0 0
- added joint elbow_31_joint: type fixed, parent shoulder_31, child elbow_31, origin xyz=0 0 0 rpy=1.5708 -1.0472 3.1416, axis 0 0 0
- added joint engine_00_joint: type fixed, parent wrist_00, child engine_00, origin xyz=1.68 0.215 0 rpy=3.1416 5.5511E-17 -1.5708, axis 0 0 0
- added joint engine_01_joint: type fixed, parent wrist_01, child engine_01, origin xyz=1.68 0.215 0 rpy=3.1416 5.5511E-17 -1.5708, axis 0 0 0
- added joint engine_10_joint: type fixed, parent wrist_10, child engine_10, origin xyz=1.68 0.215 0 rpy=3.1416 0 -1.5708, axis 0 0 0
- added joint engine_11_joint: type fixed, parent wrist_11, child engine_11, origin xyz=1.68 0.215 0 rpy=3.1416 0 -1.5708, axis 0 0 0
- added joint engine_20_joint: type fixed, parent wrist_20, child engine_20, origin xyz=1.68 0.215 0 rpy=3.1416 5.5511E-17 -1.5708, axis 0 0 0
- added joint engine_21_joint: type fixed, parent wrist_21, child engine_21, origin xyz=1.68 0.215 0 rpy=-3.1416 5.5511E-17 -1.5708, axis 0 0 0
- added joint engine_30_joint: type fixed, parent wrist_30, child engine_30, origin xyz=1.68 0.215 0 rpy=-3.1416 -3.0844E-28 -1.5708, axis 0 0 0
- added joint engine_31_joint: type fixed, parent wrist_31, child engine_31, origin xyz=1.68 0.215 0 rpy=-3.1416 -3.7076E-28 -1.5708, axis 0 0 0
- added joint shoulder_00_joint: type fixed, parent arm_0, child shoulder_00, origin xyz=2.45 0.4 0.6 rpy=-1.5708 -1.2046E-14 0, axis 0 0 0
- added joint shoulder_01_joint: type fixed, parent arm_0, child shoulder_01, origin xyz=2.45 0.4 1.1 rpy=-1.5708 -1.2046E-14 0, axis 0 0 0
- added joint shoulder_10_joint: type fixed, parent arm_1, child shoulder_10, origin xyz=2.45 0.4 0.6 rpy=-1.5708 0 0, axis 0 0 0
- added joint shoulder_11_joint: type fixed, parent arm_1, child shoulder_11, origin xyz=2.45 0.4 1.1 rpy=-1.5708 0 0, axis 0 0 0
- added joint shoulder_20_joint: type fixed, parent arm_2, child shoulder_20, origin xyz=2.45 0.4 0.6 rpy=-1.5708 -1.2046E-14 0, axis 0 0 0
- added joint shoulder_21_joint: type fixed, parent arm_2, child shoulder_21, origin xyz=2.45 0.4 1.1 rpy=-1.5708 -1.2046E-14 0, axis 0 0 0
- added joint shoulder_30_joint: type fixed, parent arm_3, child shoulder_30, origin xyz=2.45 0.4 0.6 rpy=-1.5708 0 0, axis 0 0 0
- added joint shoulder_31_joint: type fixed, parent arm_3, child shoulder_31, origin xyz=2.45 0.4 1.1 rpy=-1.5708 0 0, axis 0 0 0
- added joint top_plate_joint: type fixed, parent base_link, child top_plate, origin xyz=0.0822438122963676 0.122966095828938 0.102116404890112 rpy=1.5707963267949 0 0, axis 0 0 0
- added joint wrist_00_joint: type fixed, parent elbow_00, child wrist_00, origin xyz=-0.24651 0.64624 0 rpy=3.1416 5.5511E-17 -9.5479E-15, axis 0 0 0
- added joint wrist_01_joint: type fixed, parent elbow_01, child wrist_01, origin xyz=-0.24651 0.64624 0 rpy=3.1416 5.5511E-17 -9.5479E-15, axis 0 0 0
- added joint wrist_10_joint: type fixed, parent elbow_10, child wrist_10, origin xyz=-0.24651 0.64624 0 rpy=3.1416 0 3.1863E-14, axis 0 0 0
- added joint wrist_11_joint: type fixed, parent elbow_11, child wrist_11, origin xyz=-0.24651 0.64624 0 rpy=3.1416 0 3.1863E-14, axis 0 0 0
- added joint wrist_20_joint: type fixed, parent elbow_20, child wrist_20, origin xyz=0 -0.26928 0 rpy=-5.5511E-17 -5.5511E-17 -9.6034E-15, axis 0 0 0
- added joint wrist_21_joint: type fixed, parent elbow_21, child wrist_21, origin xyz=0.24651 0.64624 0 rpy=0 -5.5511E-17 -3.1416, axis 0 0 0
- added joint wrist_30_joint: type fixed, parent elbow_30, child wrist_30, origin xyz=0.24651 0.64624 0 rpy=0 0 3.1416, axis 0 0 0
- added joint wrist_31_joint: type fixed, parent elbow_31, child wrist_31, origin xyz=0.24651 0.64624 0 rpy=0 0 3.1416, axis 0 0 0
