Commit message: Added new model, works

File: robots/msl_skycrane.URDF (robot description, URDF)
Before this commit: robot msl_skycrane, 38 links, 37 joints
Links:
- removed link arm_0
- removed link arm_1
- removed link arm_2
- removed link arm_3
- removed link elbow_00
- removed link elbow_10
- removed link elbow_11
- removed link elbow_20
- removed link elbow_21
- removed link elbow_30
- removed link elbow_31
- removed link engine_00
- removed link engine_01
- removed link engine_10
- removed link engine_11
- removed link engine_20
- removed link engine_21
- removed link engine_30
- removed link engine_31
- removed link shoulder_00
- removed link shoulder_01
- removed link shoulder_10
- removed link shoulder_11
- removed link shoulder_20
- removed link shoulder_21
- removed link shoulder_30
- removed link shoulder_31
- removed link wrist_00
- removed link wrist_01
- removed link wrist_10
- removed link wrist_11
- removed link wrist_20
- removed link wrist_21
- removed link wrist_30
- removed link wrist_31
- added link elbow00, mass 1.7984; collision mesh filename=package://msl_skycrane_description/meshes/elbow00.STL; visual mesh filename=package://msl_skycrane_description/meshes/elbow00.STL
- added link elbow10, mass 1.7984; collision mesh filename=package://msl_skycrane_description/meshes/elbow10.STL; visual mesh filename=package://msl_skycrane_description/meshes/elbow10.STL
- added link elbow11, mass 1.7984; collision mesh filename=package://msl_skycrane_description/meshes/elbow11.STL; visual mesh filename=package://msl_skycrane_description/meshes/elbow11.STL
- added link elbow20, mass 1.7984; collision mesh filename=package://msl_skycrane_description/meshes/elbow20.STL; visual mesh filename=package://msl_skycrane_description/meshes/elbow20.STL
- added link elbow21, mass 1.7984; collision mesh filename=package://msl_skycrane_description/meshes/elbow21.STL; visual mesh filename=package://msl_skycrane_description/meshes/elbow21.STL
- added link elbow30, mass 1.7984; collision mesh filename=package://msl_skycrane_description/meshes/elbow30.STL; visual mesh filename=package://msl_skycrane_description/meshes/elbow30.STL
- added link elbow31, mass 1.7984; collision mesh filename=package://msl_skycrane_description/meshes/elbow31.STL; visual mesh filename=package://msl_skycrane_description/meshes/elbow31.STL
- added link engine00, mass 446.62; collision mesh filename=package://msl_skycrane_description/meshes/engine00.STL; visual mesh filename=package://msl_skycrane_description/meshes/engine00.STL
- added link engine01, mass 446.62; collision mesh filename=package://msl_skycrane_description/meshes/engine01.STL; visual mesh filename=package://msl_skycrane_description/meshes/engine01.STL
- added link engine10, mass 446.62; collision mesh filename=package://msl_skycrane_description/meshes/engine10.STL; visual mesh filename=package://msl_skycrane_description/meshes/engine10.STL
- added link engine11, mass 446.62; collision mesh filename=package://msl_skycrane_description/meshes/engine11.STL; visual mesh filename=package://msl_skycrane_description/meshes/engine11.STL
- added link engine20, mass 446.62; collision mesh filename=package://msl_skycrane_description/meshes/engine20.STL; visual mesh filename=package://msl_skycrane_description/meshes/engine20.STL
- added link engine21, mass 446.62; collision mesh filename=package://msl_skycrane_description/meshes/engine21.STL; visual mesh filename=package://msl_skycrane_description/meshes/engine21.STL
- added link engine30, mass 446.62; collision mesh filename=package://msl_skycrane_description/meshes/engine30.STL; visual mesh filename=package://msl_skycrane_description/meshes/engine30.STL
- added link engine31, mass 446.62; collision mesh filename=package://msl_skycrane_description/meshes/engine31.STL; visual mesh filename=package://msl_skycrane_description/meshes/engine31.STL
- added link imu_link, mass 0.001; collision box size=.01 .01 .01; visual box size=0.01 0.01 0.01
- added link shoulder00, mass 5.5908; collision mesh filename=package://msl_skycrane_description/meshes/shoulder00.STL; visual mesh filename=package://msl_skycrane_description/meshes/shoulder00.STL
- added link shoulder01, mass 5.5908; collision mesh filename=package://msl_skycrane_description/meshes/shoulder01.STL; visual mesh filename=package://msl_skycrane_description/meshes/shoulder01.STL
- added link shoulder10, mass 5.5908; collision mesh filename=package://msl_skycrane_description/meshes/shoulder10.STL; visual mesh filename=package://msl_skycrane_description/meshes/shoulder10.STL
- added link shoulder11, mass 5.5908; collision mesh filename=package://msl_skycrane_description/meshes/shoulder11.STL; visual mesh filename=package://msl_skycrane_description/meshes/shoulder11.STL
- added link shoulder20, mass 5.5908; collision mesh filename=package://msl_skycrane_description/meshes/shoulder20.STL; visual mesh filename=package://msl_skycrane_description/meshes/shoulder20.STL
- added link shoulder21, mass 5.5908; collision mesh filename=package://msl_skycrane_description/meshes/shoulder21.STL; visual mesh filename=package://msl_skycrane_description/meshes/shoulder21.STL
- added link shoulder30, mass 5.5908; collision mesh filename=package://msl_skycrane_description/meshes/shoulder30.STL; visual mesh filename=package://msl_skycrane_description/meshes/shoulder30.STL
- added link shoulder31, mass 5.5908; collision mesh filename=package://msl_skycrane_description/meshes/shoulder31.STL; visual mesh filename=package://msl_skycrane_description/meshes/shoulder31.STL
- added link suport_engine0, mass 619.74; collision mesh filename=package://msl_skycrane_description/meshes/suport_engine0.STL; visual mesh filename=package://msl_skycrane_description/meshes/suport_engine0.STL
- added link suport_engine1, mass 619.74; collision mesh filename=package://msl_skycrane_description/meshes/suport_engine1.STL; visual mesh filename=package://msl_skycrane_description/meshes/suport_engine1.STL
- added link suport_engine2, mass 619.74; collision mesh filename=package://msl_skycrane_description/meshes/suport_engine2.STL; visual mesh filename=package://msl_skycrane_description/meshes/suport_engine2.STL
- added link suport_engine3, mass 619.74; collision mesh filename=package://msl_skycrane_description/meshes/suport_engine3.STL; visual mesh filename=package://msl_skycrane_description/meshes/suport_engine3.STL
- added link wrist00, mass 1.5572; collision mesh filename=package://msl_skycrane_description/meshes/wrist00.STL; visual mesh filename=package://msl_skycrane_description/meshes/wrist00.STL
- added link wrist01, mass 1.5572; collision mesh filename=package://msl_skycrane_description/meshes/wrist01.STL; visual mesh filename=package://msl_skycrane_description/meshes/wrist01.STL
- added link wrist10, mass 1.5572; collision mesh filename=package://msl_skycrane_description/meshes/wrist10.STL; visual mesh filename=package://msl_skycrane_description/meshes/wrist10.STL
- added link wrist11, mass 1.5572; collision mesh filename=package://msl_skycrane_description/meshes/wrist11.STL; visual mesh filename=package://msl_skycrane_description/meshes/wrist11.STL
- added link wrist20, mass 1.5572; collision mesh filename=package://msl_skycrane_description/meshes/wrist20.STL; visual mesh filename=package://msl_skycrane_description/meshes/wrist20.STL
- added link wrist21, mass 1.5572; collision mesh filename=package://msl_skycrane_description/meshes/wrist21.STL; visual mesh filename=package://msl_skycrane_description/meshes/wrist21.STL
- added link wrist30, mass 1.5572; collision mesh filename=package://msl_skycrane_description/meshes/wrist30.STL; visual mesh filename=package://msl_skycrane_description/meshes/wrist30.STL
- added link wrist31, mass 1.5572; collision mesh filename=package://msl_skycrane_description/meshes/wrist31.STL; visual mesh filename=package://msl_skycrane_description/meshes/wrist31.STL
- link base_link: mass 85.813 -> 30.138
- link elbow_01: mass 3.036 -> 1.7984
- link top_plate: mass 794.77 -> 96.084
Joints:
- removed joint arm_0_joint
- removed joint arm_1_joint
- removed joint arm_2_joint
- removed joint arm_3_joint
- removed joint elbow_00_joint
- removed joint elbow_10_joint
- removed joint elbow_11_joint
- removed joint elbow_20_joint
- removed joint elbow_21_joint
- removed joint elbow_30_joint
- removed joint elbow_31_joint
- removed joint engine_00_joint
- removed joint engine_01_joint
- removed joint engine_10_joint
- removed joint engine_11_joint
- removed joint engine_20_joint
- removed joint engine_21_joint
- removed joint engine_30_joint
- removed joint engine_31_joint
- removed joint shoulder_00_joint
- removed joint shoulder_01_joint
- removed joint shoulder_10_joint
- removed joint shoulder_11_joint
- removed joint shoulder_20_joint
- removed joint shoulder_21_joint
- removed joint shoulder_30_joint
- removed joint shoulder_31_joint
- removed joint wrist_00_joint
- removed joint wrist_01_joint
- removed joint wrist_10_joint
- removed joint wrist_11_joint
- removed joint wrist_20_joint
- removed joint wrist_21_joint
- removed joint wrist_30_joint
- removed joint wrist_31_joint
- added joint elbow00_joint: type fixed, parent shoulder00, child elbow00, origin xyz=0.0299999999999998 0 0.301961524227067 rpy=1.57079632679489 1.0471975511966 2.20934381900405E-14, axis 0 0 0
- added joint elbow10_joint: type fixed, parent shoulder10, child elbow10, origin xyz=0.0299999999999998 0 0.301961524227067 rpy=1.5707963267949 1.04719755119661 0, axis 0 0 0
- added joint elbow11_joint: type fixed, parent shoulder11, child elbow11, origin xyz=0.0300000000000002 0 0.301961524227067 rpy=1.5707963267949 1.04719755119661 0, axis 0 0 0
- added joint elbow20_joint: type fixed, parent shoulder20, child elbow20, origin xyz=0.203205080756887 0 0.401961524227066 rpy=-1.5707963267949 1.04719755119661 2.20934381900412E-14, axis 0 0 0
- added joint elbow21_joint: type fixed, parent shoulder21, child elbow21, origin xyz=-0.406410161513767 -0.500000000000006 -0.234641016151378 rpy=1.5707963267949 -1.0471975511966 -3.14159265358977, axis 0 0 0
- added joint elbow30_joint: type fixed, parent shoulder30, child elbow30, origin xyz=0.0299999999999998 0 0.301961524227067 rpy=1.5707963267949 -1.04719755119661 3.14159265358979, axis 0 0 0
- added joint elbow31_joint: type fixed, parent shoulder31, child elbow31, origin xyz=0.0299999999999994 0 0.301961524227066 rpy=1.5707963267949 -1.04719755119661 3.14159265358979, axis 0 0 0
- added joint engine00_joint: type fixed, parent wrist00, child engine00, origin xyz=1.68 0.214999999999989 0 rpy=-3.14159265358979 5.55111512312578E-17 -1.57079632679492, axis 0 0 0
- added joint engine01_joint: type fixed, parent wrist01, child engine01, origin xyz=1.68 0.214999999999988 0 rpy=-3.14159265358979 5.55111512312578E-17 -1.57079632679492, axis 0 0 0
- added joint engine10_joint: type fixed, parent wrist10, child engine10, origin xyz=1.68 0.214999999999996 0 rpy=3.14159265358979 0 -1.57079632679489, axis 0 0 0
- added joint engine11_joint: type fixed, parent wrist11, child engine11, origin xyz=1.68 0.215000000000003 0 rpy=3.14159265358979 0 -1.57079632679489, axis 0 0 0
- added joint engine20_joint: type fixed, parent wrist20, child engine20, origin xyz=1.68 0.214999999999989 0 rpy=-3.14159265358979 5.55111512312578E-17 -1.57079632679492, axis 0 0 0
- added joint engine21_joint: type fixed, parent wrist21, child engine21, origin xyz=1.68 0.214999999999988 0 rpy=-3.14159265358979 5.55111512312578E-17 -1.57079632679492, axis 0 0 0
- added joint engine30_joint: type fixed, parent wrist30, child engine30, origin xyz=1.68 0.214999999999997 0 rpy=-3.14159265358978 -3.08444613941416E-28 -1.57079632679489, axis 0 0 0
- added joint engine31_joint: type fixed, parent wrist31, child engine31, origin xyz=1.68 0.215 0 rpy=-3.1416 -3.7076E-28 -1.5708, axis 0 0 0
- added joint imu_joint: type fixed, parent base_link, child imu_link, origin xyz=0 0 -1.5, axis 1 0 0
- added joint shoulder00_joint: type fixed, parent suport_engine0, child shoulder00, origin xyz=1.95 0.4 0.59999999999999 rpy=-1.5707963267949 -1.20459198171829E-14 0, axis 0 0 0
- added joint shoulder01_joint: type fixed, parent suport_engine0, child shoulder01, origin xyz=1.95000000000001 0.399999999999999 1.09999999999999 rpy=-1.5707963267949 -1.20459198171829E-14 0, axis 0 0 0
- added joint shoulder10_joint: type fixed, parent suport_engine1, child shoulder10, origin xyz=1.95 0.399999999999999 0.6 rpy=-1.5707963267949 0 0, axis 0 0 0
- added joint shoulder11_joint: type fixed, parent suport_engine1, child shoulder11, origin xyz=1.95 0.399999999999999 1.1 rpy=-1.5707963267949 0 0, axis 0 0 0
- added joint shoulder20_joint: type fixed, parent suport_engine2, child shoulder20, origin xyz=1.95 0.399999999999999 0.59999999999999 rpy=-1.5707963267949 -1.20459198171829E-14 0, axis 0 0 0
- added joint shoulder21_joint: type fixed, parent suport_engine2, child shoulder21, origin xyz=2.38641016151378 0.936602540378443 0.599999999999988 rpy=-1.5707963267949 -1.20459198171829E-14 0, axis 0 0 0
- added joint shoulder30_joint: type fixed, parent suport_engine3, child shoulder30, origin xyz=1.95000000000002 0.399999999999999 0.599999999999943 rpy=-1.5707963267949 0 0, axis 0 0 0
- added joint shoulder31_joint: type fixed, parent suport_engine3, child shoulder31, origin xyz=1.95000000000003 0.399999999999999 1.09999999999994 rpy=-1.5707963267949 0 0, axis 0 0 0
- added joint suport_engine0_joint: type fixed, parent top_plate, child suport_engine0, origin xyz=-0.1116 -2 -1.5067 rpy=0 1.0472 0, axis 0 0 0
- added joint suport_engine1_joint: type fixed, parent top_plate, child suport_engine1, origin xyz=1.2490381056767 -2 -0.849999999999998 rpy=0 0 0, axis 0 0 0
- added joint suport_engine2_joint: type fixed, parent top_plate, child suport_engine2, origin xyz=0.111602540378529 -2 1.50669872981077 rpy=3.14159265358979 -1.04719755119662 3.14159265358979, axis 0 0 0
- added joint suport_engine3_joint: type fixed, parent top_plate, child suport_engine3, origin xyz=-1.24903810567659 -2 0.850000000000035 rpy=3.14159265358979 0 3.14159265358979, axis 0 0 0
- added joint wrist00_joint: type fixed, parent elbow00, child wrist00, origin xyz=0 0.469282032302756 0 rpy=3.14159265358979 5.55111512312578E-17 -9.54791801177635E-15, axis 0 0 0
- added joint wrist01_joint: type fixed, parent elbow_01, child wrist01, origin xyz=0 0.469282032302755 0 rpy=3.14159265358979 5.55111512312578E-17 -9.54791801177635E-15, axis 0 0 0
- added joint wrist10_joint: type fixed, parent elbow10, child wrist10, origin xyz=0 0.469282032302755 0 rpy=3.14159265358979 0 9.6034291630076E-15, axis 0 0 0
- added joint wrist11_joint: type fixed, parent elbow11, child wrist11, origin xyz=0 0.469282032302754 0 rpy=3.14159265358979 0 9.6034291630076E-15, axis 0 0 0
- added joint wrist20_joint: type fixed, parent elbow20, child wrist20, origin xyz=0 -0.269282032302755 0 rpy=-5.55111512312578E-17 -5.55111512312578E-17 -9.6034291630076E-15, axis 0 0 0
- added joint wrist21: type fixed, parent elbow21, child wrist21, origin xyz=0 0.469282032302756 0 rpy=0 -5.55111512312578E-17 -3.14159265358978, axis 0 0 0
- added joint wrist30_joint: type fixed, parent elbow30, child wrist30, origin xyz=0 0.469282032302755 0 rpy=0 0 3.14159265358978, axis 0 0 0
- added joint wrist31_joint: type fixed, parent elbow31, child wrist31, origin xyz=0 0.469282032302755 0 rpy=0 0 3.14159265358978, axis 0 0 0
- joint elbow_01_joint: origin xyz=0 0 0 rpy=1.5708 1.0472 2.2093E-14 -> xyz=0.0299999999999994 0 0.301961524227067 rpy=1.57079632679489 1.0471975511966 2.20934381900405E-14; parent shoulder_01 -> shoulder01
- joint top_plate_joint: origin xyz=0.0822438122963676 0.122966095828938 0.102116404890112 rpy=1.5707963267949 0 0 -> xyz=0.082244 0.12297 0.10212 rpy=1.5708 0 0

File: robots/msl_skycrane_description.xacro (robot description, xacro)
@@ -1,4 +1,4 @@
 <?xml version="1.0"?>
 <robot xmlns:xacro="http://ros.org/wiki/xacro" name="msl_skycrane_description">
-    <!-- <xacro:include filename="$(find msl_skycrane_description)/robot/landing_engines.xacro"/> -->
+    <xacro:include filename="$(find msl_skycrane_description)/robots/msl_skycrane.URDF" />
 </robot>
