Commit message: update

File: robots/landing_engines.xacro (robot description, xacro)
@@ -1,3 +1,2 @@
-<?xml version="1.0"?>
 <?xml version="1.0"?>
 <robot xmlns:xacro="http://ros.org/wiki/xacro" name="msl_skycrane_description">

File: robots/msl_skycrane.URDF (robot description, URDF)
Before this commit: robot msl_skycrane_description, 39 links, 38 joints
Links:
- link elbow00: geometry collision mesh filename=package://msl_skycrane_description/meshes/elbow.STL; visual mesh filename=package://msl_skycrane_description/meshes/elbow.STL
- link elbow10: geometry collision mesh filename=package://msl_skycrane_description/meshes/elbow.STL; visual mesh filename=package://msl_skycrane_description/meshes/elbow.STL
- link elbow11: geometry collision mesh filename=package://msl_skycrane_description/meshes/elbow.STL; visual mesh filename=package://msl_skycrane_description/meshes/elbow.STL
- link elbow20: geometry collision mesh filename=package://msl_skycrane_description/meshes/elbow.STL; visual mesh filename=package://msl_skycrane_description/meshes/elbow.STL
- link elbow21: geometry collision mesh filename=package://msl_skycrane_description/meshes/elbow.STL; visual mesh filename=package://msl_skycrane_description/meshes/elbow.STL
- link elbow30: geometry collision mesh filename=package://msl_skycrane_description/meshes/elbow.STL; visual mesh filename=package://msl_skycrane_description/meshes/elbow.STL
- link elbow31: geometry collision mesh filename=package://msl_skycrane_description/meshes/elbow.STL; visual mesh filename=package://msl_skycrane_description/meshes/elbow.STL
- link elbow_01: geometry collision mesh filename=package://msl_skycrane_description/meshes/elbow.STL; visual mesh filename=package://msl_skycrane_description/meshes/elbow.STL
- link engine00: geometry collision mesh filename=package://msl_skycrane_description/meshes/engine.STL; visual mesh filename=package://msl_skycrane_description/meshes/engine.STL
- link engine01: geometry collision mesh filename=package://msl_skycrane_description/meshes/engine.STL; visual mesh filename=package://msl_skycrane_description/meshes/engine.STL
- link engine10: geometry collision mesh filename=package://msl_skycrane_description/meshes/engine.STL; visual mesh filename=package://msl_skycrane_description/meshes/engine.STL
- link engine11: geometry collision mesh filename=package://msl_skycrane_description/meshes/engine.STL; visual mesh filename=package://msl_skycrane_description/meshes/engine.STL
- link engine20: geometry collision mesh filename=package://msl_skycrane_description/meshes/engine.STL; visual mesh filename=package://msl_skycrane_description/meshes/engine.STL
- link engine21: geometry collision mesh filename=package://msl_skycrane_description/meshes/engine.STL; visual mesh filename=package://msl_skycrane_description/meshes/engine.STL
- link engine30: geometry collision mesh filename=package://msl_skycrane_description/meshes/engine.STL; visual mesh filename=package://msl_skycrane_description/meshes/engine.STL
- link engine31: geometry collision mesh filename=package://msl_skycrane_description/meshes/engine.STL; visual mesh filename=package://msl_skycrane_description/meshes/engine.STL
- link suport_engine0: geometry collision mesh filename=package://msl_skycrane_description/meshes/suport_engine.STL; visual mesh filename=package://msl_skycrane_description/meshes/suport_engine.STL
- link suport_engine1: geometry collision mesh filename=package://msl_skycrane_description/meshes/suport_engine.STL; visual mesh filename=package://msl_skycrane_description/meshes/suport_engine.STL
- link suport_engine2: geometry collision mesh filename=package://msl_skycrane_description/meshes/suport_engine.STL; visual mesh filename=package://msl_skycrane_description/meshes/suport_engine.STL
- link suport_engine3: geometry collision mesh filename=package://msl_skycrane_description/meshes/suport_engine.STL; visual mesh filename=package://msl_skycrane_description/meshes/suport_engine.STL
- link wrist00: geometry collision mesh filename=package://msl_skycrane_description/meshes/wrist.STL; visual mesh filename=package://msl_skycrane_description/meshes/wrist.STL
- link wrist01: geometry collision mesh filename=package://msl_skycrane_description/meshes/wrist.STL; visual mesh filename=package://msl_skycrane_description/meshes/wrist.STL
- link wrist10: geometry collision mesh filename=package://msl_skycrane_description/meshes/wrist.STL; visual mesh filename=package://msl_skycrane_description/meshes/wrist.STL
- link wrist11: geometry collision mesh filename=package://msl_skycrane_description/meshes/wrist.STL; visual mesh filename=package://msl_skycrane_description/meshes/wrist.STL
- link wrist20: geometry collision mesh filename=package://msl_skycrane_description/meshes/wrist.STL; visual mesh filename=package://msl_skycrane_description/meshes/wrist.STL
- link wrist21: geometry collision mesh filename=package://msl_skycrane_description/meshes/wrist.STL; visual mesh filename=package://msl_skycrane_description/meshes/wrist.STL
- link wrist30: geometry collision mesh filename=package://msl_skycrane_description/meshes/wrist.STL; visual mesh filename=package://msl_skycrane_description/meshes/wrist.STL
- link wrist31: geometry collision mesh filename=package://msl_skycrane_description/meshes/wrist.STL; visual mesh filename=package://msl_skycrane_description/meshes/wrist.STL
Joints:
- joint imu_joint: origin xyz=0 0 -1.5 -> xyz=0 0 -2 rpy=0 0 0
